File: kicad_files/kicad_win.kicad_pcb (KiCad board)
At the start: 2 copper layers, 68.6 x 53.3 mm, 9 parts, among them P1 Power, P2 Analog, P3 Digital, P4 Digital, P5 CONN_01X01, P6 CONN_01X01, P7 CONN_01X01, P8 CONN_01X01

Commit message: new version of the schematic
Parts:
- added BZ1: Device_Buzzer, Buzzers_Beepers:Buzzer_12x9.5RM7.6, F.Cu at (128.4, 102.6)
- added C1: C, Capacitors_THT:CP_Radial_D5.0mm_P2.50mm, F.Cu at (174.9, 104.4)
- added C2: C, Capacitors_THT:CP_Radial_D5.0mm_P2.50mm, F.Cu at (188.1, 112.9)
- added C3: C, Capacitors_THT:CP_Radial_D5.0mm_P2.50mm, F.Cu at (188.1, 106.3)
- added C4: C, Capacitors_THT:CP_Radial_D5.0mm_P2.50mm, F.Cu at (127.8, 92.2)
- added C5: C, Capacitors_THT:CP_Radial_D5.0mm_P2.50mm, F.Cu at (188.2, 99.8)
- added C6: C, Capacitors_THT:CP_Radial_D5.0mm_P2.50mm, F.Cu at (181.5, 104.4)
- added C7: C, Capacitors_THT:CP_Radial_D5.0mm_P2.50mm, F.Cu at (174.9, 110.9)
- added D1: LED, LEDs_THT:LED_D5.0mm, F.Cu at (188.5, 92.7)
- added R10: R, Resistors_THT:R_Axial_DIN0207_L6.3mm_D2.5mm_P10.16mm_Horizontal, F.Cu at (147.7, 111.2)
- added R11: R, Resistors_THT:R_Axial_DIN0207_L6.3mm_D2.5mm_P10.16mm_Horizontal, F.Cu at (161.0, 99.1)
- added R12: R, Resistors_THT:R_Axial_DIN0207_L6.3mm_D2.5mm_P10.16mm_Horizontal, F.Cu at (174.3, 95.0)
- added R13: R, Resistors_THT:R_Axial_DIN0207_L6.3mm_D2.5mm_P10.16mm_Horizontal, F.Cu at (161.0, 103.1)
- added R14: R, Resistors_THT:R_Axial_DIN0207_L6.3mm_D2.5mm_P10.16mm_Horizontal, F.Cu at (161.0, 107.2)
- added R15: R, Resistors_THT:R_Axial_DIN0207_L6.3mm_D2.5mm_P10.16mm_Horizontal, F.Cu at (161.0, 111.2)
- added R16: R, Resistors_THT:R_Axial_DIN0207_L6.3mm_D2.5mm_P10.16mm_Horizontal, F.Cu at (147.7, 91.0)
- added R2: R, Resistors_THT:R_Axial_DIN0207_L6.3mm_D2.5mm_P10.16mm_Horizontal, F.Cu at (147.7, 95.0)
- added R3: R, Resistors_THT:R_Axial_DIN0207_L6.3mm_D2.5mm_P10.16mm_Horizontal, F.Cu at (161.0, 91.0)
- added R4: R, Resistors_THT:R_Axial_DIN0207_L6.3mm_D2.5mm_P10.16mm_Horizontal, F.Cu at (147.7, 99.1)
- added R5: R, Resistors_THT:R_Axial_DIN0207_L6.3mm_D2.5mm_P10.16mm_Horizontal, F.Cu at (174.3, 99.1)
- added R6: R, Resistors_THT:R_Axial_DIN0207_L6.3mm_D2.5mm_P10.16mm_Horizontal, F.Cu at (161.0, 95.0)
- added R7: R, Resistors_THT:R_Axial_DIN0207_L6.3mm_D2.5mm_P10.16mm_Horizontal, F.Cu at (147.7, 103.1)
- added R8: R, Resistors_THT:R_Axial_DIN0207_L6.3mm_D2.5mm_P10.16mm_Horizontal, F.Cu at (147.7, 107.2)
- added R9: R, Resistors_THT:R_Axial_DIN0207_L6.3mm_D2.5mm_P10.16mm_Horizontal, F.Cu at (174.3, 91.0)
- added U1: AD8001AR, LTC1050ACN8:PDIP-8_N, F.Cu at (171.4, 68.4)
- added U2: AD8001AR, LTC1050ACN8:PDIP-8_N, F.Cu at (170.4, 80.1)
- added U3: AD8001AR, LTC1050ACN8:PDIP-8_N, F.Cu at (181.4, 68.4)
- added U4: Gas_Sensor_TO-5-10, Package_TO_SOT_THT:TO-5-10, F.Cu at (174.1, 76.0)
Connections:
- P1 pad 1: Net-(P1-Pad1) -> (no net)
- P1 pad 2: /IOREF -> (no net)
- P1 pad 3: /Reset -> (no net)
- P1 pad 8: /Vin -> (no net)
- P2 pad 3: /A2 -> (no net)
- P2 pad 4: /A3 -> (no net)
- P2 pad 5: /A4(SDA) -> (no net)
- P2 pad 6: /A5(SCL) -> (no net)
- P3 pad 1: /A5(SCL) -> (no net)
- P3 pad 10: /8 -> (no net)
- P3 pad 2: /A4(SDA) -> (no net)
- P3 pad 3: /AREF -> (no net)
- P3 pad 6: /12(MISO) -> (no net)
- P3 pad 7: /11(**/MOSI) -> (no net)
- P3 pad 8: /10(**/SS) -> (no net)
- P4 pad 1: /7 -> (no net)
- P4 pad 4: /4 -> (no net)
- P4 pad 7: /1(Tx) -> (no net)
- P4 pad 8: /0(Rx) -> (no net)
- P5 pad 1: Net-(P5-Pad1) -> (no net)
- P6 pad 1: Net-(P6-Pad1) -> (no net)
- P7 pad 1: Net-(P7-Pad1) -> (no net)
- P8 pad 1: Net-(P8-Pad1) -> (no net)
Routing:
- net (no net): track 0.00 -> 170.2 mm
- net /A4(SDA): track 88.1 -> 0.00 mm
- net /A5(SCL): track 82.1 -> 0.00 mm

Commit message: Complete electronic circuits
Parts:
- added MODULE1: RN2483-I_RM095, RN2483-I_RM095:MICROCHIP_RN2483-I%2fRM095, B.Cu at (141.5, 90.2)
- moved C3 72.1 mm to (116.1, 108.6), turned to 90 degrees
- moved R5 61.1 mm to (113.5, 92.7)
- moved U2 58.7 mm to (120.5, 111.1), turned to 270 degrees
- moved R9 57.4 mm to (123.7, 118.1), turned to 180 degrees
- moved C2 57.0 mm to (131.9, 122.6), turned to 180 degrees
- moved U4 53.2 mm to (139.6, 116.4), turned to 180 degrees
- moved C1 48.2 mm to (128.1, 92.7), turned to 90 degrees
- moved U3 45.2 mm to (157.4, 106.7), turned to 90 degrees
- moved R6 37.8 mm to (123.7, 101.0), turned to 180 degrees
- moved R7 34.8 mm to (113.5, 96.5)
- moved R8 34.8 mm to (113.5, 113.7)
- moved D1 34.5 mm to (154.2, 95.2), turned to 90 degrees
- moved C4 33.5 mm to (113.6, 122.6)
- moved C5 32.8 mm to (155.4, 101.0), turned to 180 degrees
- moved R16 29.5 mm to (175.1, 80.0), turned to 180 degrees
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Connections:
- P3 pad 2: (no net) -> /9(**)
- P3 pad 5: /13LED(SCK) -> (no net)
- P3 pad 6: (no net) -> /12(MISO)
- P3 pad 7: (no net) -> /11(**/MOSI)
- P3 pad 8: (no net) -> /10(**/SS)
- R1 pad 2: /13LED(SCK) -> /2
Routing:
- net (no net): track 170.2 -> 0.00 mm
- net +5V: track 0.00 -> 91.0 mm
- net /A1: track 0.00 -> 62.5 mm
- net /2: track 0.00 -> 53.8 mm
- net GND: track 56.3 -> 3.81 mm
- net /Heater: track 0.00 -> 49.8 mm
- net Net-(C1-Pad1): track 0.00 -> 42.7 mm
- net /9(**): track 0.00 -> 32.3 mm
- net +3V3: track 0.00 -> 28.5 mm
- net /12(MISO): track 0.00 -> 26.6 mm
- net Net-(C3-Pad2): track 0.00 -> 25.4 mm
- net Net-(C3-Pad1): track 0.00 -> 24.6 mm
- net /Gas_Temp_Target_Anal: track 0.00 -> 22.5 mm
- net /13LED(SCK): track 19.3 -> 0.00 mm
- net /Gas_Trigger_Offset_Anal: track 0.00 -> 17.8 mm
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- added copper zone on B.Cu, net GND
Other:
- board text added: "Romain Saboret Noël Taillardat SMART GAS SENSOR 2019"

Commit message: probably final
Parts:
- C1, C2, C4: value C -> 100n
- C3: value C -> 1u
- C5, C6, C7: value C -> 10u
- PT3: renamed from R12; value R -> 1k
- PT4: renamed from R10; value R -> 10k
- R1, R13, R4, R9: value R -> 1k
- R11, R14, R15, R16, R2: value R -> 10k
- R5, R8: value R -> 100k
- R6: value R -> 500
- renumbered R7 to PT1, R3 to PT2
Connections:
- MODULE1 pad 10: (no net) -> Net-(MODULE1-Pad10)
- MODULE1 pad 12: (no net) -> +3V3
- MODULE1 pad 13: (no net) -> Net-(MODULE1-Pad13)
- MODULE1 pad 14: (no net) -> Net-(MODULE1-Pad14)
- MODULE1 pad 2: (no net) -> Net-(MODULE1-Pad2)
- MODULE1 pad 23: (no net) -> Net-(MODULE1-Pad23)
- MODULE1 pad 25: (no net) -> Net-(MODULE1-Pad25)
- MODULE1 pad 3: (no net) -> Net-(MODULE1-Pad3)
- MODULE1 pad 30: (no net) -> Net-(MODULE1-Pad30)
- MODULE1 pad 31: (no net) -> Net-(MODULE1-Pad31)
- MODULE1 pad 34: (no net) -> +3V3
- MODULE1 pad 35: (no net) -> Net-(MODULE1-Pad35)
- MODULE1 pad 36: (no net) -> Net-(MODULE1-Pad36)
- MODULE1 pad 37: (no net) -> Net-(MODULE1-Pad37)
- MODULE1 pad 38: (no net) -> Net-(MODULE1-Pad38)
- MODULE1 pad 39: (no net) -> Net-(MODULE1-Pad39)
- MODULE1 pad 4: (no net) -> Net-(MODULE1-Pad4)
- MODULE1 pad 40: (no net) -> Net-(MODULE1-Pad40)
- MODULE1 pad 43: (no net) -> Net-(MODULE1-Pad43)
- MODULE1 pad 44: (no net) -> Net-(MODULE1-Pad44)
- MODULE1 pad 45: (no net) -> Net-(MODULE1-Pad45)
- MODULE1 pad 46: (no net) -> Net-(MODULE1-Pad46)
- MODULE1 pad 5: (no net) -> Net-(MODULE1-Pad5)
- MODULE1 pad 9: (no net) -> Net-(MODULE1-Pad9)
- P1 pad 1: (no net) -> Net-(P1-Pad1)
- P1 pad 2: (no net) -> /IOREF
- P1 pad 3: (no net) -> /Reset
- P1 pad 8: (no net) -> /Vin
- P2 pad 3: (no net) -> /A2
- P2 pad 4: (no net) -> /A3
- P2 pad 5: (no net) -> /A4(SDA)
- P2 pad 6: (no net) -> /A5(SCL)
- P3 pad 1: (no net) -> Net-(P3-Pad1)
- P3 pad 10: (no net) -> /8
- P3 pad 3: (no net) -> /AREF
- P3 pad 5: (no net) -> /13LED(SCK)
- P4 pad 1: (no net) -> /7
- P4 pad 4: (no net) -> /4
- P4 pad 7: (no net) -> /1(Tx)
- P4 pad 8: (no net) -> /0(Rx)
- P5 pad 1: (no net) -> Net-(P5-Pad1)
- P6 pad 1: (no net) -> Net-(P6-Pad1)
- P7 pad 1: (no net) -> Net-(P7-Pad1)
- P8 pad 1: (no net) -> Net-(P8-Pad1)
- PT2 pad 1: Net-(R3-Pad1) -> /A1
- R4 pad 1: /A1 -> Net-(R4-Pad1)
- R4 pad 2: Net-(R3-Pad1) -> /A1
- U1 pad 1: (no net) -> Net-(U1-Pad1)
- U1 pad 2: /A1 -> Net-(R4-Pad1)
- U1 pad 5: (no net) -> Net-(U1-Pad5)
- U1 pad 8: (no net) -> Net-(U1-Pad8)
- U2 pad 1: (no net) -> Net-(U2-Pad1)
- U2 pad 5: (no net) -> Net-(U2-Pad5)
- U2 pad 8: (no net) -> Net-(U2-Pad8)
- U3 pad 1: (no net) -> Net-(U3-Pad1)
- U3 pad 5: (no net) -> Net-(U3-Pad5)
- U3 pad 7: +5V -> +3V3
- U3 pad 8: (no net) -> Net-(U3-Pad8)
Routing:
- net +3V3: track 28.5 -> 95.0 mm
- net Net-(R4-Pad1): track 0.00 -> 26.3 mm
- net /A1: track 62.5 -> 43.6 mm
- net Net-(R3-Pad1): track 3.70 -> 0.00 mm
- net +5V: track 91.0 -> 87.9 mm
