File: kicad_files/kicad_win.sch (KiCad schematic (older format))
At the start: 30 parts, among them P1 Power, P2 Analog, P3 Digital, P4 Digital, P5 CONN_01X01, P6 CONN_01X01, P7 CONN_01X01, P8 CONN_01X01

Commit message: lul
Connections:
- net labels added: Buzzer
- net labels removed: Gas_Temp
Other:
- note added: "El buzz"
Changed lines of the file:
@@
 	1    0    0    -1
 $EndComp
-Text Label 7600 3600 0    50   ~ 0
-Vin
 $Comp
 L kicad_win-rescue:R-Device R?
@@
 Gas_Trigger_Diff
 Text Label 8900 2600 2    50   ~ 0
-Gas_Temp
+Poly_Resistor
 Text Label 10550 1900 0    50   ~ 0
 Lora_TX
@@
 Text Label 8750 5200 2    50   ~ 0
 Gas_Value
+Text Label 10550 2000 0    50   ~ 0
+Buzzer
+Text Label 6600 3250 2    50   ~ 0
+Buzzer
+$Comp
+L kicad_win-rescue:GND-power #PWR?
+U 1 1 5DEA192E
+P 6600 3450
+F 0 "#PWR?" H 6600 3200 50  0001 C CNN
+F 1 "GND" H 6600 3300 50  0000 C CNN
+F 2 "" H 6600 3450 50  0000 C CNN
+F 3 "" H 6600 3450 50  0000 C CNN
+	1    6600 3450
+	0    1    1    0
+$EndComp
+Wire Notes Line
+	6200 3000 7450 3000
+Wire Notes Line
+	7450 3000 7450 3600
+Wire Notes Line
+	6200 3000 6200 3600
+Wire Notes Line
+	6200 3600 7450 3600
+Text Notes 6250 3100 0    50   ~ 0
+El buzz
+Wire Notes Line
+	6600 3000 6600 3150
+Wire Notes Line
+	6600 3150 6200 3150
 $EndSCHEMATC

Commit message: new version of the schematic
Parts:
- removed U? (x3): LTC1050, LTC1050CN8:PDIP-8_N, symbol kicad_win-rescue:LTC1100xN8-Amplifier_Instrumentation
- added C5, C6, C7: C, Capacitors_THT:CP_Radial_D5.0mm_P2.50mm, symbol kicad_win-rescue:C-Device
- added R14, R15, R16: R, Resistors_THT:R_Axial_DIN0207_L6.3mm_D2.5mm_P10.16mm_Horizontal, symbol kicad_win-rescue:R-Device
- added U1, U2, U3: AD8001AR, LTC1050ACN8:PDIP-8_N, symbol Amplifier_Operational:AD8001AR
- added U4: Gas_Sensor_TO-5-10, Package_TO_SOT_THT:TO-5-10, symbol Gas_Sensor:Gas_Sensor_TO-5-10
- BZ1: renamed from BZ?; footprint Buzzers_Beepers:BUZZER -> Buzzers_Beepers:Buzzer_12x9.5RM7.6
- D1: footprint LEDs:LED_D5.0mm -> LEDs_THT:LED_D5.0mm
- gave numbers to parts that had none: 16
Connections:
- net labels added: GasSens, Gas_Temp_Target_Anal, Gas_Temp_Target_PWM, Gas_Trigger_Diff_Anal, Gas_Trigger_Diff_PWM, Gas_Trigger_Offset_Anal, Gas_Trigger_Offset_PWM, TempSens
- net labels removed: Gas_Temp_Target, Gas_Trigger_Diff, Gas_Trigger_Offset, Poly_Resistor
- wire segments 94 -> 96
Other:
- note added: "DACs"
- note added: "L'ao peut délivrer assez ? \nou faut mettre ca dans un transistor"
- note added: "Sensor"
- moved on the sheet: R10, R11, R12, R13

Commit message: Complete electronic circuits
Parts:
- added MODULE1: RN2483-I_RM095, RN2483-I_RM095:MICROCHIP_RN2483-I%2fRM095, symbol RN2483-I_RM095:RN2483-I_RM095
Connections:
- net 10(**/SS): now also MODULE1.6 (UART_TX)
- net 11(**/MOSI): now also MODULE1.7 (UART_RX)
- net 12(MISO): now also MODULE1.32 (~RESET~)
- net 13LED(SCK): no longer R1.2
- net 2: now also R1.2
- net 9(**): now also P3.2 (Pin_2)
- net GND: now also MODULE1.1 (GND), MODULE1.11 (GND), MODULE1.20 (GND), MODULE1.21 (GND), MODULE1.22 (GND), MODULE1.24 (GND), MODULE1.26 (GND), MODULE1.27 (GND), MODULE1.28 (GND), MODULE1.33 (GND), MODULE1.41 (GND), MODULE1.47 (GND), MODULE1.8 (GND)
Other:
- moved on the sheet: BZ1, C1, C2, C3, C4, D1, R1, R10, R11, R12, R13, R2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

Commit message: probably final
Parts:
- C1, C2, C4: value C -> 100n
- C3: value C -> 1u
- C5, C6, C7: value C -> 10u
- PT3: renamed from R12; value R -> 1k
- PT4: renamed from R10; value R -> 10k
- R1, R13, R4, R9: value R -> 1k
- R11, R14, R15, R16, R2: value R -> 10k
- R5, R8: value R -> 100k
- R6: value R -> 500
- U1, U2, U3: symbol Amplifier_Operational:AD8001AR -> kicad_win-rescue:AD8001AR-Amplifier_Operational
- renumbered R7 to PT1, R3 to PT2
Connections:
- net +3V3: now also MODULE1.12 (VDD1), MODULE1.34 (VDD2), U3.7 (V+)
- net +5V: no longer U3.7 (V+)
- net A1: now also PT2.1, R4.2; no longer R4.1, U1.2 (-)
- new net: R4.1, U1.2 (-)
Other:
- moved on the sheet: R4
Changed lines of the file:
@@
 EESchema Schematic File Version 4
 LIBS:kicad_win-cache
-EELAYER 30 0
+EELAYER 29 0
 EELAYER END
 $Descr A4 11693 8268
@@
 P 7550 2000
 F 0 "R1" V 7757 2000 50  0000 C CNN
-F 1 "R" V 7666 2000 50  0000 C CNN
+F 1 "1k" V 7666 2000 50  0000 C CNN
 F 2 "Resistors_THT:R_Axial_DIN0207_L6.3mm_D2.5mm_P10.16mm_Horizontal" V 7665 2000 50  0001 C CNN
 F 3 "~" H 7550 2000 50  0001 C CNN
@@
 Text Label 5600 3500 2    50   ~ 0
 Gas_Temp_Target_Anal
-Text Label 5350 3900 2    50   ~ 0
+Text Label 4950 3900 2    50   ~ 0
 TempSens
-$Comp
-L kicad_win-rescue:R-Device R4
-U 1 1 5DE1BEC5
-P 5250 3700
-F 0 "R4" V 5150 3650 50  0000 C CNN
-F 1 "R" V 5150 3750 50  0000 C CNN
-F 2 "Resistors_THT:R_Axial_DIN0207_L6.3mm_D2.5mm_P10.16mm_Horizontal" V 5365 3700 50  0001 C CNN
-F 3 "~" H 5250 3700 50  0001 C CNN
-	1    5250 3700
-	0    1    1    0
-$EndComp
-Wire Wire Line
-	5600 3700 5400 3700
+Wire Wire Line
+	5600 3700 5550 3700
 $Comp
 L kicad_win-rescue:+5V-power #PWR0110
@@
 	4750 3700 4800 3700
 $Comp
-L kicad_win-rescue:R-Device R3
+L kicad_win-rescue:R-Device PT2
 U 1 1 5DE2933A
 P 4950 3700
-F 0 "R3" V 4850 3650 50  0000 C CNN
+F 0 "PT2" V 4850 3650 50  0000 C CNN
 F 1 "R" V 4850 3750 50  0000 C CNN
 F 2 "Resistors_THT:R_Axial_DIN0207_L6.3mm_D2.5mm_P10.16mm_Horizontal" V 5065 3700 50  0001 C CNN
@@
 	5400 3150 4450 3150
 Wire Wire Line
-	5600 3700 5600 3900
-$Comp
-L kicad_win-rescue:+5V-power #PWR0113
-U 1 1 5DE474A2
-P 2450 1500
-F 0 "#PWR0113" H 2450 1350 50  0001 C CNN
-F 1 "+5V" H 2465 1673 50  0000 C CNN
-F 2 "" H 2450 1500 50  0001 C CNN
-F 3 "" H 2450 1500 50  0001 C CNN
-	1    2450 1500
-	1    0    0    -1
-$EndComp
-Wire Wire Line
 	2450 2100 2450 2150
 $Comp
@@
 P 3050 1500
 F 0 "R13" H 3150 1450 50  0000 C CNN
-F 1 "R" H 3150 1550 50  0000 C CNN
+F 1 "1k" H 3150 1550 50  0000 C CNN
 F 2 "Resistors_THT:R_Axial_DIN0207_L6.3mm_D2.5mm_P10.16mm_Horizontal" V 3165 1500 50  0001 C CNN
 F 3 "~" H 3050 1500 50  0001 C CNN
@@
 $EndComp
 $Comp
-L kicad_win-rescue:R-Device R12
+L kicad_win-rescue:R-Device PT3
 U 1 1 5DE5F3AC
 P 3050 950
-F 0 "R12" H 3150 900 50  0000 C CNN
-F 1 "R" H 3150 1000 50  0000 C CNN
+F 0 "PT3" H 3150 900 50  0000 C CNN
+F 1 "1k" H 3150 1000 50  0000 C CNN
 F 2 "Resistors_THT:R_Axial_DIN0207_L6.3mm_D2.5mm_P10.16mm_Horizontal" V 3165 950 50  0001 C CNN
 F 3 "~" H 3050 950 50  0001 C CNN
@@
 P 2500 1200
 F 0 "R11" V 2707 1200 50  0000 C CNN
-F 1 "R" V 2616 1200 50  0000 C CNN
+F 1 "10k" V 2616 1200 50  0000 C CNN
 F 2 "Resistors_THT:R_Axial_DIN0207_L6.3mm_D2.5mm_P10.16mm_Horizontal" V 2615 1200 50  0001 C CNN
 F 3 "~" H 2500 1200 50  0001 C CNN
@@
 	2050 1200 2350 1200
 $Comp
-L kicad_win-rescue:R-Device R10
+L kicad_win-rescue:R-Device PT4
 U 1 1 5DE70C6E
 P 1750 1700
-F 0 "R10" V 1957 1700 50  0000 C CNN
-F 1 "R" V 1866 1700 50  0000 C CNN
+F 0 "PT4" V 1957 1700 50  0000 C CNN
+F 1 "10k" V 1866 1700 50  0000 C CNN
 F 2 "Resistors_THT:R_Axial_DIN0207_L6.3mm_D2.5mm_P10.16mm_Horizontal" V 1865 1700 50  0001 C CNN
 F 3 "~" H 1750 1700 50  0001 C CNN
@@
 $EndComp
 $Comp
-L power:GND #PWR0102
+L kicad_win-rescue:GND-power #PWR0102
 U 1 1 5DE52EC9
 P 8000 1250
@@
 P 5150 950
 F 0 "R14" V 5050 900 50  0000 C CNN
-F 1 "R" V 5050 1000 50  0000 C CNN
+F 1 "10k" V 5050 1000 50  0000 C CNN
 F 2 "Resistors_THT:R_Axial_DIN0207_L6.3mm_D2.5mm_P10.16mm_Horizontal" V 5265 950 50  0001 C CNN
 F 3 "~" H 5150 950 50  0001 C CNN
@@
 P 5400 1100
 F 0 "C5" H 5515 1146 50  0000 L CNN
-F 1 "C" H 5515 1055 50  0000 L CNN
+F 1 "10u" H 5515 1055 50  0000 L CNN
 F 2 "Capacitors_THT:CP_Radial_D5.0mm_P2.50mm" H 5438 950 50  0001 C CNN
 F 3 "~" H 5400 1100 50  0001 C CNN
@@
 Connection ~ 5400 950
 $Comp
-L power:GND #PWR0116
+L kicad_win-rescue:GND-power #PWR0116
 U 1 1 5DE75256
 P 5400 1250
@@
 P 5150 1550
 F 0 "R15" V 5050 1500 50  0000 C CNN
-F 1 "R" V 5050 1600 50  0000 C CNN
+F 1 "10k" V 5050 1600 50  0000 C CNN
 F 2 "Resistors_THT:R_Axial_DIN0207_L6.3mm_D2.5mm_P10.16mm_Horizontal" V 5265 1550 50  0001 C CNN
 F 3 "~" H 5150 1550 50  0001 C CNN
@@
 P 5400 1700
 F 0 "C6" H 5515 1746 50  0000 L CNN
-F 1 "C" H 5515 1655 50  0000 L CNN
+F 1 "10u" H 5515 1655 50  0000 L CNN
 F 2 "Capacitors_THT:CP_Radial_D5.0mm_P2.50mm" H 5438 1550 50  0001 C CNN
 F 3 "~" H 5400 1700 50  0001 C CNN
@@
 Connection ~ 5400 1550
 $Comp
-L power:GND #PWR0117
+L kicad_win-rescue:GND-power #PWR0117
 U 1 1 5DE7CB54
 P 5400 1850
@@
 P 5150 2150
 F 0 "R16" V 5050 2100 50  0000 C CNN
-F 1 "R" V 5050 2200 50  0000 C CNN
+F 1 "10k" V 5050 2200 50  0000 C CNN
 F 2 "Resistors_THT:R_Axial_DIN0207_L6.3mm_D2.5mm_P10.16mm_Horizontal" V 5265 2150 50  0001 C CNN
 F 3 "~" H 5150 2150 50  0001 C CNN
@@
 P 5400 2300
 F 0 "C7" H 5515 2346 50  0000 L CNN
-F 1 "C" H 5515 2255 50  0000 L CNN
+F 1 "10u" H 5515 2255 50  0000 L CNN
 F 2 "Capacitors_THT:CP_Radial_D5.0mm_P2.50mm" H 5438 2150 50  0001 C CNN
 F 3 "~" H 5400 2300 50  0001 C CNN
@@
 Connection ~ 5400 2150
 $Comp
-L power:GND #PWR0118
+L kicad_win-rescue:GND-power #PWR0118
 U 1 1 5DE8050D
 P 5400 2450
@@
 GasSens
 $Comp
-L power:+3.3V #PWR0119
+L kicad_win-rescue:+3.3V-power #PWR0119
 U 1 1 5DEA8961
 P 7900 1100
@@
 Gas_Trigger_Offset_Anal
 Wire Wire Line
-	5350 3900 5600 3900
+	4950 3900 5200 3900
 Connection ~ 2050 1700
 Wire Notes Line
@@
 	7200 700  7200 850
 $Comp
-L Amplifier_Operational:AD8001AR U3
+L kicad_win-rescue:AD8001AR-Amplifier_Operational U3
 U 1 1 5DEFD374
 P 2550 1800
@@
 $EndComp
 $Comp
-L Amplifier_Operational:AD8001AR U1
+L kicad_win-rescue:AD8001AR-Amplifier_Operational U1
 U 1 1 5DF098E8
 P 5900 3600
@@
 	1    0    0    -1
 $EndComp
-Connection ~ 5600 3700
 Wire Wire Line
 	7450 4100 7450 4250
@@
 	8900 4700 9050 4700
 $Comp
-L Amplifier_Operational:AD8001AR U2
+L kicad_win-rescue:AD8001AR-Amplifier_Operational U2
 U 1 1 5DE466C8
 P 8750 4700
@@
 P 9200 4200
 F 0 "C2" H 9315 4246 50  0000 L CNN
-F 1 "C" H 9315 4155 50  0000 L CNN
+F 1 "100n" H 9315 4155 50  0000 L CNN
 F 2 "Capacitors_THT:CP_Radial_D5.0mm_P2.50mm" H 9238 4050 50  0001 C CNN
 F 3 "~" H 9200 4200 50  0001 C CNN
@@
 P 7450 4850
 F 0 "C1" H 7565 4896 50  0000 L CNN
-F 1 "C" H 7565 4805 50  0000 L CNN
+F 1 "100n" H 7565 4805 50  0000 L CNN
 F 2 "Capacitors_THT:CP_Radial_D5.0mm_P2.50mm" H 7488 4700 50  0001 C CNN
 F 3 "~" H 7450 4850 50  0001 C CNN
@@
 P 10100 4700
 F 0 "R9" V 10307 4700 50  0000 C CNN
-F 1 "R" V 10216 4700 50  0000 C CNN
+F 1 "1k" V 10216 4700 50  0000 C CNN
 F 2 "Resistors_THT:R_Axial_DIN0207_L6.3mm_D2.5mm_P10.16mm_Horizontal" V 10215 4700 50  0001 C CNN
 F 3 "~" H 10100 4700 50  0001 C CNN
@@
 P 10400 4950
 F 0 "C4" H 10515 4996 50  0000 L CNN
-F 1 "C" H 10515 4905 50  0000 L CNN
+F 1 "100n" H 10515 4905 50  0000 L CNN
 F 2 "Capacitors_THT:CP_Radial_D5.0mm_P2.50mm" H 10438 4800 50  0001 C CNN
 F 3 "~" H 10400 4950 50  0001 C CNN
@@
 P 9800 4950
 F 0 "R8" H 9650 4900 50  0000 C CNN
-F 1 "R" H 9650 5000 50  0000 C CNN
+F 1 "100k" H 9650 5000 50  0000 C CNN
 F 2 "Resistors_THT:R_Axial_DIN0207_L6.3mm_D2.5mm_P10.16mm_Horizontal" V 9915 4950 50  0001 C CNN
 F 3 "~" H 9800 4950 50  0001 C CNN
@@
 $EndComp
 $Comp
-L kicad_win-rescue:R-Device R7
+L kicad_win-rescue:R-Device PT1
 U 1 1 5DD74FA9
 P 8300 5800
-F 0 "R7" H 8150 5750 50  0000 C CNN
+F 0 "PT1" H 8150 5750 50  0000 C CNN
 F 1 "R" H 8150 5850 50  0000 C CNN
 F 2 "Resistors_THT:R_Axial_DIN0207_L6.3mm_D2.5mm_P10.16mm_Horizontal" V 8415 5800 50  0001 C CNN
@@
 P 7850 4850
 F 0 "R5" H 7700 4800 50  0000 C CNN
-F 1 "R" H 7700 4900 50  0000 C CNN
+F 1 "100k" H 7700 4900 50  0000 C CNN
 F 2 "Resistors_THT:R_Axial_DIN0207_L6.3mm_D2.5mm_P10.16mm_Horizontal" V 7965 4850 50  0001 C CNN
 F 3 "~" H 7850 4850 50  0001 C CNN
@@
 P 8300 5450
 F 0 "R6" H 8150 5400 50  0000 C CNN
-F 1 "R" H 8150 5500 50  0000 C CNN
+F 1 "500" H 8150 5500 50  0000 C CNN
 F 2 "Resistors_THT:R_Axial_DIN0207_L6.3mm_D2.5mm_P10.16mm_Horizontal" V 8415 5450 50  0001 C CNN
 F 3 "~" H 8300 5450 50  0001 C CNN
@@
 P 7450 4400
 F 0 "R2" H 7300 4350 50  0000 C CNN
-F 1 "R" H 7300 4450 50  0000 C CNN
+F 1 "10k" H 7300 4450 50  0000 C CNN
 F 2 "Resistors_THT:R_Axial_DIN0207_L6.3mm_D2.5mm_P10.16mm_Horizontal" V 7565 4400 50  0001 C CNN
 F 3 "~" H 7450 4400 50  0001 C CNN
@@
 P 9450 4950
 F 0 "C3" H 9565 4996 50  0000 L CNN
-F 1 "C" H 9565 4905 50  0000 L CNN
+F 1 "1u" H 9565 4905 50  0000 L CNN
 F 2 "Capacitors_THT:CP_Radial_D5.0mm_P2.50mm" H 9488 4800 50  0001 C CNN
 F 3 "~" H 9450 4950 50  0001 C CNN
@@
 $EndComp
 $Comp
-L power:GND #PWR0120
+L kicad_win-rescue:GND-power #PWR0120
 U 1 1 5DED76D9
 P 3200 5650
@@
 Text Label 10550 1300 0    50   ~ 0
 Buzzer
+$Comp
+L kicad_win-rescue:+3.3V-power #PWR?
+U 1 1 5E286648
+P 2450 1500
+F 0 "#PWR?" H 2450 1350 50  0001 C CNN
+F 1 "+3.3V" V 2450 1750 50  0000 C CNN
+F 2 "" H 2450 1500 50  0000 C CNN
+F 3 "" H 2450 1500 50  0000 C CNN
+	1    2450 1500
+	1    0    0    -1
+$EndComp
+$Comp
+L kicad_win-rescue:+3.3V-power #PWR?
+U 1 1 5E289E71
+P 3200 3200
+F 0 "#PWR?" H 3200 3050 50  0001 C CNN
+F 1 "+3.3V" V 3200 3450 50  0000 C CNN
+F 2 "" H 3200 3200 50  0000 C CNN
+F 3 "" H 3200 3200 50  0000 C CNN
+	1    3200 3200
+	1    0    0    -1
+$EndComp
+Wire Wire Line
+	3200 3200 3200 3300
+Connection ~ 3200 3200
+Wire Wire Line
+	5250 3700 5200 3700
+Wire Wire Line
+	5200 3700 5200 3900
+Connection ~ 5200 3700
+Wire Wire Line
+	5200 3700 5100 3700
+$Comp
+L kicad_win-rescue:R-Device R4
+U 1 1 5DE1BEC5
+P 5400 3700
+F 0 "R4" V 5300 3650 50  0000 C CNN
+F 1 "1k" V 5300 3800 50  0000 C CNN
+F 2 "Resistors_THT:R_Axial_DIN0207_L6.3mm_D2.5mm_P10.16mm_Horizontal" V 5515 3700 50  0001 C CNN
+F 3 "~" H 5400 3700 50  0001 C CNN
+	1    5400 3700
+	0    1    1    0
+$EndComp
 $EndSCHEMATC
